File: kicad/Nucleo64_Z80.kicad_sch (KiCad schematic)
At the start: 9 parts, among them U2 AS6C4008-55PCN, U3 Z80CPU

Commit message: Add Nucleo64_Z80 PCB revision 1.0
Parts:
- removed JP1, JP2: SolderJumper_2_Open, Jumper:SolderJumper-2_P1.3mm_Open_RoundedPad1.0x1.5mm, symbol Jumper:SolderJumper_2_Open
- added JP1, JP2: SolderJumper_3_Bridged12, Jumper:SolderJumper-3_P1.3mm_Bridged12_RoundedPad1.0x1.5mm_NumberLabels, symbol Jumper:SolderJumper_3_Bridged12
- added JP4: SolderJumper_2_Open, Jumper:SolderJumper-2_P1.3mm_Open_RoundedPad1.0x1.5mm, symbol Jumper:SolderJumper_2_Open
- added JP5, JP6: SolderJumper_2_Bridged, Jumper:SolderJumper-2_P1.3mm_Bridged_RoundedPad1.0x1.5mm, symbol Jumper:SolderJumper_2_Bridged
- C1, C2: value C_Small -> 0.1uF
- R1: value R_Small -> 200
Connections:
- net A13: now also U1.CN10_23 (PA_8); no longer U1.CN7_23 (PC_13)
- net A14: now also U1.CN10_21 (PA_9); no longer U1.CN7_25 (PC_14)
- net A15: now also U1.CN10_33 (PA_10); no longer U1.CN7_27 (PC_15)
- net A16: now also JP5.2 (B)
- net A17: now also JP6.2 (B)
- net BANK_SEL0: now also JP5.1 (A)
- net BANK_SEL1: now also JP6.1 (A)
- net GND: now also U2.1 (A18)
- net SPI1_SCLK: now also U1.CN10_11 (PA_5); no longer U1.CN10_31 (PB_3)
- net VCC: now also JP2.1 (A)
- net ~{INT}: now also JP2.2 (C); no longer U1.CN10_11 (PA_5)
- net ~{M1}: now also JP3.2 (B); no longer U1.CN7_30 (PA_1)
- net ~{RFSH}: now also JP4.2 (B); no longer U1.CN10_21 (PA_9)
- net ~{SPI1_SS}: now also JP1.2 (C); no longer U1.CN7_32 (PA_4)
- net ~{WAIT}: now also U1.CN7_30 (PA_1); no longer U1.CN10_33 (PA_10)
- removed net A18: JP3.2 (B), U2.1 (A18)
- net BANK_SEL2 renamed PC13
- net PC13: now also U1.CN7_23 (PC_13); no longer U1.CN10_23 (PA_8)
- new net PA4: JP1.1 (A), U1.CN7_32 (PA_4)
- new net PB3: JP1.3 (B), U1.CN10_31 (PB_3)
- new net PC14: JP2.3 (B), U1.CN7_25 (PC_14)
- new net PC15: JP4.1 (A), U1.CN7_27 (PC_15)
Other:
- title: (none) -> Nucleo64 Z80
- moved on the sheet: R1
